File: DoDecaCharlieCylonCR2032.brd (EAGLE design)
At the start: 40.6 x 33 mm, 20 parts, among them J1 AVR_SPI, U1 TINY85

Commit message: changing logo
Parts:
- U$1: value 18 USC 707 -> USER_HACKABLE; device 4h:4H_LOGO_6 -> logo:USER_HACKABLE
Other:
- board text added: "User Hackable"
- board text added: "userhackable.com"
- board text removed: "Cache Makers"
- board text removed: "cachemakers.org"
Changed lines of the file:
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@@
 <hole x="36.83" y="29.21" drill="3.81"/>
 <text x="30.1625" y="14.9225" size="0.6096" layer="21" rot="R90" align="center">PULL-UP</text>
-<text x="22.5425" y="9.2075" size="1.778" layer="21" align="center">Cache Makers</text>
-<text x="22.5425" y="7.3025" size="1.016" layer="21" align="center">cachemakers.org</text>
+<text x="22.5425" y="9.2075" size="1.778" layer="21" align="center">User Hackable</text>
+<text x="22.5425" y="7.3025" size="1.016" layer="21" align="center">userhackable.com</text>
 <text x="10.16" y="29.21" size="1.016" layer="21" align="center">Cap
 Sense</text>
@@
 <attribute name="VALUE" x="31.75" y="17.145" size="0.8128" layer="21" font="vector" ratio="15" rot="R270" align="center-left"/>
 </element>
-<element name="U$1" library="4h" package="4H_LOGO_6" value="18 USC 707" x="20.32" y="20.32"/>
 <element name="R2" library="SparkFun-Sensors" package="PHOTOCELL" value="PHOTOCELLPTH" x="3.81" y="23.495" smashed="yes" rot="R270"/>
+<element name="U$1" library="logo" package="USER_HACKABLE" value="USER_HACKABLE" x="20.32" y="20.32"/>
 </elements>
 <signals>
