File: DoDecaCharlieCylonCR2032.brd (EAGLE design)
At the start: 40.6 x 33 mm, 20 parts, among them J1 AVR_SPI, U1 TINY85

Commit message: changing branding
Parts:
- U$1: value USER_HACKABLE -> 18 USC 707; device logo:USER_HACKABLE -> 4h:4H_LOGO_6
Other:
- board text added: "Cache Makers"
- board text added: "cachemakers.org"
- board text removed: "User Hackable"
- board text removed: "userhackable.com"
Changed lines of the file:
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@@
 <hole x="36.83" y="29.21" drill="3.81"/>
 <text x="30.1625" y="14.9225" size="0.6096" layer="21" rot="R90" align="center">PULL-UP</text>
-<text x="22.5425" y="9.2075" size="1.778" layer="21" align="center">User Hackable</text>
-<text x="22.5425" y="7.3025" size="1.016" layer="21" align="center">userhackable.com</text>
+<text x="22.5425" y="9.2075" size="1.778" layer="21" align="center">Cache Makers</text>
+<text x="22.5425" y="7.3025" size="1.016" layer="21" align="center">cachemakers.org</text>
 <text x="10.16" y="29.21" size="1.016" layer="21" align="center">Cap
 Sense</text>
@@
 <element name="LED12" library="barbary_enterprises" package="LED-OVAL" value="" x="37.7825" y="3.81" rot="R90"/>
 <element name="S1" library="barbary_enterprises" package="TACTILE-PTH" value="" x="36.83" y="20.32" smashed="yes" rot="R90"/>
-<element name="U$3" library="battery" package="CR2032-THRU" value="" x="20.32" y="23.1775" rot="MR0"/>
+<element name="U$3" library="battery" package="CR2032-THRU" value="" x="20.32" y="23.1775" smashed="yes" rot="MR0">
+<attribute name="VALUE" x="24.638" y="16.8275" size="1.6764" layer="28" font="vector" rot="MR0"/>
+</element>
 <element name="R1" library="barbary_enterprises" package="AXIAL-0.3" value="1M" x="31.75" y="14.9225" smashed="yes" rot="R270">
 <attribute name="VALUE" x="31.75" y="17.145" size="0.8128" layer="21" font="vector" ratio="15" rot="R270" align="center-left"/>
 </element>
+<element name="U$1" library="4h" package="4H_LOGO_6" value="18 USC 707" x="20.32" y="20.32"/>
 <element name="R2" library="SparkFun-Sensors" package="PHOTOCELL" value="PHOTOCELLPTH" x="3.81" y="23.495" smashed="yes" rot="R270"/>
-<element name="U$1" library="logo" package="USER_HACKABLE" value="USER_HACKABLE" x="20.32" y="20.32"/>
 </elements>
 <signals>

Commit message: updating logo
Parts:
- U$1: value 18 USC 707 -> USER_HACKABLE; device 4h:4H_LOGO_6 -> logo:USER_HACKABLE
Changed lines of the file:
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@@
 <element name="LED12" library="barbary_enterprises" package="LED-OVAL" value="" x="37.7825" y="3.81" rot="R90"/>
 <element name="S1" library="barbary_enterprises" package="TACTILE-PTH" value="" x="36.83" y="20.32" smashed="yes" rot="R90"/>
-<element name="U$3" library="battery" package="CR2032-THRU" value="" x="20.32" y="23.1775" smashed="yes" rot="MR0">
-<attribute name="VALUE" x="24.638" y="16.8275" size="1.6764" layer="28" font="vector" rot="MR0"/>
-</element>
+<element name="U$3" library="battery" package="CR2032-THRU" value="" x="20.32" y="23.1775" rot="MR0"/>
 <element name="R1" library="barbary_enterprises" package="AXIAL-0.3" value="1M" x="31.75" y="14.9225" smashed="yes" rot="R270">
 <attribute name="VALUE" x="31.75" y="17.145" size="0.8128" layer="21" font="vector" ratio="15" rot="R270" align="center-left"/>
 </element>
-<element name="U$1" library="4h" package="4H_LOGO_6" value="18 USC 707" x="20.32" y="20.32"/>
 <element name="R2" library="SparkFun-Sensors" package="PHOTOCELL" value="PHOTOCELLPTH" x="3.81" y="23.495" smashed="yes" rot="R270"/>
+<element name="U$1" library="logo" package="USER_HACKABLE" value="USER_HACKABLE" x="20.32" y="20.32"/>
 </elements>
 <signals>
