File: DoDecaCharlieCylonCR2032.brd (EAGLE design)
At the start: 40.6 x 33 mm, 20 parts, among them J1 AVR_SPI, U1 TINY85

Commit message: updating schematic
Routing:
- net VCC: track 49.5 -> 50.4 mm
Changed lines of the file:
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@@
 <wire x1="12.065" y1="14.2875" x2="12.065" y2="15.875" width="0.8128" layer="16"/>
 <wire x1="12.065" y1="15.875" x2="9.525" y2="18.415" width="0.8128" layer="16"/>
-<wire x1="9.525" y1="18.415" x2="9.525" y2="20.6375" width="0.8128" layer="16"/>
-<wire x1="9.525" y1="20.6375" x2="9.525" y2="23.0505" width="0.8128" layer="16"/>
+<wire x1="9.525" y1="18.415" x2="9.525" y2="23.0505" width="0.8128" layer="16"/>
 <wire x1="9.525" y1="23.0505" x2="9.652" y2="23.1775" width="0.8128" layer="16"/>
-<wire x1="5.08" y1="19.05" x2="6.985" y2="20.955" width="0.8128" layer="16"/>
-<wire x1="6.985" y1="20.955" x2="9.2075" y2="20.955" width="0.8128" layer="16"/>
-<wire x1="9.2075" y1="20.955" x2="9.525" y2="20.6375" width="0.8128" layer="16"/>
+<wire x1="5.08" y1="19.05" x2="9.2075" y2="23.1775" width="0.8128" layer="1"/>
+<wire x1="9.2075" y1="23.1775" x2="9.652" y2="23.1775" width="0.8128" layer="1"/>
 </signal>
 <signal name="N$2">

Commit message: updating schematic
Parts:
- U$1: value USER_HACKABLE -> (none); device logo:USER_HACKABLE -> 4h:4H_LOGO_6
Changed lines of the file:
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@@
 </element>
 <element name="R2" library="SparkFun-Sensors" package="PHOTOCELL" value="PHOTOCELLPTH" x="3.81" y="23.495" smashed="yes" rot="R270"/>
-<element name="U$1" library="logo" package="USER_HACKABLE" value="USER_HACKABLE" x="20.32" y="20.32"/>
+<element name="U$1" library="4h" package="4H_LOGO_6" value="" x="20.32" y="20.32"/>
 </elements>
 <signals>
