File: DoDecaCharlieCylonCR2032.sch (EAGLE design)
At the start: 20 parts, among them J1 AVR_SPI, U1 TINY85

Commit message: changing logo
Parts:
- U$1: value 18 USC 707 -> USER_HACKABLE; device 4h:4H-LOGO6 -> logo:USER_HACKABLE
Changed lines of the file:
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@@
 <part name="R1" library="barbary_enterprises" deviceset="RESISTOR" device="AXIAL-0.3" value="1M"/>
 <part name="GND4" library="SparkFun-Aesthetics" deviceset="GND" device=""/>
-<part name="U$1" library="4h" deviceset="4H-LOGO" device="6" value="18 USC 707"/>
 <part name="R2" library="SparkFun-Sensors" deviceset="PHOTOCELL" device="PTH"/>
+<part name="U$1" library="logo" deviceset="USER_HACKABLE" device=""/>
 </parts>
 <sheets>
@@
 <instance part="R1" gate="G$1" x="78.74" y="40.64" rot="R270"/>
 <instance part="GND4" gate="1" x="78.74" y="10.16"/>
+<instance part="R2" gate="G$1" x="78.74" y="22.86" rot="R90"/>
 <instance part="U$1" gate="G$1" x="124.46" y="25.4"/>
-<instance part="R2" gate="G$1" x="78.74" y="22.86" rot="R90"/>
 </instances>
 <busses>
