File: DoDecaCharlieCylonCR2032.sch (EAGLE design)
At the start: 20 parts, among them J1 AVR_SPI, U1 TINY85

Commit message: updating logo
Changed lines of the file:
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@@
 <instance part="GND4" gate="1" x="78.74" y="10.16"/>
 <instance part="R2" gate="G$1" x="78.74" y="22.86" rot="R90"/>
-<instance part="U$1" gate="G$1" x="124.46" y="25.4"/>
+<instance part="U$1" gate="G$1" x="121.92" y="25.4"/>
 </instances>
 <busses>

Commit message: updating schematic
Parts:
- U$1: value USER_HACKABLE -> (none); device logo:USER_HACKABLE -> 4h:4H-LOGO6
Changed lines of the file:
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@@
 <part name="GND4" library="SparkFun-Aesthetics" deviceset="GND" device=""/>
 <part name="R2" library="SparkFun-Sensors" deviceset="PHOTOCELL" device="PTH"/>
-<part name="U$1" library="logo" deviceset="USER_HACKABLE" device=""/>
+<part name="U$1" library="4h" deviceset="4H-LOGO" device="6"/>
 </parts>
 <sheets>
@@
 <instance part="GND4" gate="1" x="78.74" y="10.16"/>
 <instance part="R2" gate="G$1" x="78.74" y="22.86" rot="R90"/>
-<instance part="U$1" gate="G$1" x="121.92" y="25.4"/>
+<instance part="U$1" gate="G$1" x="139.7" y="27.94"/>
 </instances>
 <busses>
